File: RP2350B_board.kicad_sch (KiCad schematic)
At the start: 44 parts, among them IC1 W25Q128JVSIM, IC2 UA78M33CDCYG3, J1 USB_C_Receptacle_USB2.0_16P, J2 SWD, J3 Conn_01x25_Pin, J4 Conn_01x25_Pin, J5 Conn_01x25_Pin, J6 Conn_01x25_Pin, J7 Conn_01x25_Pin, J8 Conn_01x25_Pin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

Commit message: refactor: start new layout
Signed-off-by: Aditya Agarwal <aditya.agarwal030504@gmail.com>
Parts:
- removed C1, C2, C3, C5: 4.7u, Capacitor_SMD:C_0402_1005Metric, symbol Device:C
- removed C10, C11, C12, C13, C14, C15, C16, C19, C20, C4, C6, C7, C8, C9: 100n, Capacitor_SMD:C_0402_1005Metric, symbol Device:C
- removed C17, C18: 15p, Capacitor_SMD:C_0402_1005Metric, symbol Device:C
- removed IC1: W25Q128JVSIM, W25Q128JVSIM:SOIC127P790X216-8N, symbol W25Q128JVSIM:W25Q128JVSIM
- removed IC2: UA78M33CDCYG3, UA78M33CDCYG3:SOT230P700X180-4N, symbol UA78M33CDCYG3:UA78M33CDCYG3
- removed J1: USB_C_Receptacle_USB2.0_16P, Connector_USB:USB_C_Receptacle_GCT_USB4105-xx-A_16P_TopMnt_Horizontal, symbol Connector:USB_C_Receptacle_USB2.0_16P
- removed J2: SWD, Connector_PinHeader_2.54mm:PinHeader_1x04_P2.54mm_Vertical, symbol Connector:Conn_01x04_Pin
- removed J3, J4, J5, J6, J7, J8: Conn_01x25_Pin, Connector_PinHeader_2.54mm:PinHeader_1x25_P2.54mm_Vertical, symbol Connector:Conn_01x25_Pin
- removed L1: 3.3u, Inductor_SMD:L_0603_1608Metric, symbol Device:L
- removed R1: 33, Resistor_SMD:R_0402_1005Metric, symbol Device:R
- removed R2, R3: 5.1K, Resistor_SMD:R_0402_1005Metric, symbol Device:R
- removed R5: 0, Resistor_SMD:R_0402_1005Metric, symbol Device:R
- removed R6: DNF, Resistor_SMD:R_0402_1005Metric, symbol Device:R
- removed R7, R8, R9: 1K, Resistor_SMD:R_0402_1005Metric, symbol Device:R
- removed S2: PTS636_SM43_LFS, PTS636SM43LFS, symbol PTS636_SM43_LFS:PTS636_SM43_LFS
- removed Y1: ABM8-272-T3, ABM8-272-T3:ABM8272T3, symbol ABM8-272-T3:ABM8-272-T3
- R4: value 10K -> 1K
Connections:
- net GND: now also R4.1; no longer U1.62 (VREG_PGND)
- net XOUT: now reaches U1.31 (XOUT)
- net XIN: now reaches U1.30 (XIN)
- net at S1.2 (NO): now also R4.2
- net +1V1 renamed DVDD
- net DVDD: no longer U1.65 (VREG_FB)
- net +3.3v renamed IOVDD
- net IOVDD: no longer R4.2, U1.64 (VREG_VIN)
- new net VREG_FB: U1.65 (VREG_FB)
- new net VREG_PGND: U1.62 (VREG_PGND)
- new net VREG_VIN: U1.64 (VREG_VIN)
- no-connect marks 2 -> 0
Other:
- added sheet Clock (clock.kicad_sch)
- added sheet Connectors (Connectors.kicad_sch)
- added sheet Flash (flash.kicad_sch)
- added sheet Power (power.kicad_sch)
- note added: "Reset Switch"
- note removed: "RP2350 Development Board"
- company: (none) -> Dumblebots
- title: (none) -> RP2350B Development Board
